Commit message: Avancement de la simulation

File: src/sara_description/urdf/sara.urdf (robot description, URDF)
Before this commit: robot SARA, 11 links, 10 joints
Links:
- removed link clavicule_link
- removed link fixLowerArm_link
- removed link fixUpperArm_link
- removed link gripper_link
- removed link laser_link
- removed link rotLowerArm_link
- removed link rotUpperArm_link
- added link base_laser_link, mass 0.5; collision cylinder length=0.1 radius=0.03; visual cylinder length=0.1 radius=0.03
- added link camera_link, mass 0.5; visual box size=0.02 0.2 0.01
- link base_link: mass None -> 10; geometry collision box size=0.65 0.55 0.57; collision box size=0.65 0.78 0.14
- link head_link: mass None -> 5; geometry collision box size=0.25 0.1 0.4; collision sphere radius=0.2
- link neck_link: mass None -> 2; geometry visual box size=0.11 0.11 0.11
- link torso_link: mass None -> 10; geometry collision box size=0.4 0.4 0.2; collision box size=0.8 0.2 0.2
Joints:
- removed joint WristRot_joint
- removed joint Wrist_joint
- removed joint elbow_joint
- removed joint shoulderRot_joint
- removed joint shoulder_joint
- removed joint sternoclavicular_joint
- added joint camera_joint: type fixed, parent head_link, child camera_link, origin xyz=-0.09 0.075 0 rpy=0 3.14 -1.57, axis 0 0 1
- joint laser_joint: child laser_link -> base_laser_link; origin xyz=0 0.14 0.14 rpy=0 0 0 -> xyz=0 0.14 0.19 rpy=0 0 1.57
- joint neckHead_joint: limit lower=-1.04 upper=1.04 effort=1000.0 velocity=0.5 -> lower=-0.40 upper=1.04 effort=1000.0 velocity=0.5; origin xyz=0 0 0.2 rpy=0 1.57 0 -> xyz=0 0 0.11 rpy=0 1.57 0; type revolute -> fixed
- joint spine_joint: axis 0 0 1.4 -> 0 0 1; limit lower=1 upper=1.5 effort=1000.0 velocity=0.2 -> lower=0 upper=0.5 effort=1000.0 velocity=0.2; origin xyz=0 0 0 rpy=0 0 0 -> xyz=0 0 1 rpy=0 0 0; type prismatic -> fixed
- joint torsoNeck_joint: origin xyz=0 0 0.2 rpy=0 0 0 -> xyz=0 0 0.09 rpy=0 0 0; type revolute -> fixed

Commit message: NAVsss et URDF du bras

File: src/sara_description/urdf/sara.urdf (robot description, URDF)
Before this commit: robot SARA, 6 links, 5 joints
Links:
- added link clavicule_link; collision mesh filename=package://sara_description/meshes/1-epaule.STL scale=0.001 0.001 0.001; visual mesh filename=package://sara_description/meshes/1-epaule.STL scale=0.001 0.001 0.001
- added link fixLowerArm_link; collision mesh filename=package://sara_description/meshes/4-coude.STL scale=0.001 0.001 0.001; visual mesh filename=package://sara_description/meshes/4-coude.STL scale=0.001 0.001 0.001
- added link fixUpperArm_link; collision mesh filename=package://sara_description/meshes/1-epaule.STL scale=0.001 0.001 0.001; visual mesh filename=package://sara_description/meshes/1-epaule.STL scale=0.001 0.001 0.001
- added link rotLowerArm_link; collision mesh filename=package://sara_description/meshes/5-pince-avant-bras.STL scale=0.001 0.001 0.001; visual mesh filename=package://sara_description/meshes/5-pince-avant-bras.STL scale=0.001 0.001 0.001
- added link rotUpperArm_link; collision mesh filename=package://sara_description/meshes/3-bras_haut.STL scale=0.001 0.001 0.001; visual mesh filename=package://sara_description/meshes/3-bras_haut.STL scale=0.001 0.001 0.001
- added link spine_link, mass 10; visual cylinder length=0.9 radius=0.04
- link base_link: geometry collision box size=0.55 0.64311 0.57; collision box size=0.7637 0.64311 0.14
- link head_link: geometry collision box size=0.02 0.16 0.31; collision sphere radius=0.1
- link torso_link: geometry collision box size=0.04 0.38 0.075; collision box size=0.18 0.18 0.28
Joints:
- removed joint spine_joint
- added joint WristRot_joint: type revolute, parent fixLowerArm_link, child rotLowerArm_link, origin xyz=0.0945 0 0 rpy=0 1.57 0, axis 0 0 1, limit lower=-3.1416 upper=3.1416 effort=1000.0 velocity=0.5
- added joint base_spine_joint: type fixed, parent base_link, child spine_link, origin xyz=0.2 0 0 rpy=0 0 0, axis 0 0 1
- added joint elbow_joint: type revolute, parent rotUpperArm_link, child fixLowerArm_link, origin xyz=0 0 0.31 rpy=3.1416 -1.57 0, axis 0 0 1, limit lower=-2.23 upper=2 effort=1000.0 velocity=0.5
- added joint shoulderRot_joint: type revolute, parent fixUpperArm_link, child rotUpperArm_link, origin xyz=0.085 0 0 rpy=0 1.57 0, axis 0 0 1, limit lower=-3.1416 upper=3.1416 effort=1000.0 velocity=0.5
- added joint shoulder_joint: type revolute, parent clavicule_link, child fixUpperArm_link, origin xyz=0.085 0 0 rpy=1.57 0 1.57, axis 0 0 1, limit lower=-3.1416 upper=3.1416 effort=1000.0 velocity=0.5
- added joint spine_torso_joint: type fixed, parent spine_link, child torso_link, origin xyz=0 0 1 rpy=0 0 0, axis 0 0 1, limit lower=0 upper=0.5 effort=1000.0 velocity=0.2
- added joint sternoclavicular_joint: type revolute, parent torso_link, child clavicule_link, origin xyz=0 -0.145 0 rpy=-1.57 0 -1.57, axis 0 0 1, limit lower=-1.57 upper=1.57 effort=1000.0 velocity=0.5
- joint camera_joint: axis 0 0 1 -> 0 1 0; origin xyz=-0.09 0.075 0 rpy=0 3.14 -1.57 -> xyz=0.075 -0.09 0 rpy=1.57 0 0
- joint laser_joint: origin xyz=0 0.14 0.19 rpy=0 0 1.57 -> xyz=0.34 0 0.19 rpy=0 0 0
- joint neckHead_joint: origin xyz=0 0 0.11 rpy=0 1.57 0 -> xyz=0 0 0.11 rpy=-1.57 0 0

Commit message: update to sara.urdf

File: src/sara_description/urdf/sara.urdf (robot description, URDF)
Before this commit: robot SARA, 12 links, 11 joints
Links:
- removed link base_link
- added link sara_base, mass 10; collision box size=0.55 0.64311 0.57; collision box size=0.7637 0.64311 0.14
Joints:
- joint WristRot_joint: origin xyz=0.0945 0 0 rpy=0 1.57 0 -> xyz=0 0.0945 0 rpy=1.5708 0 0
- joint base_spine_joint: parent base_link -> sara_base
- joint elbow_joint: origin xyz=0 0 0.31 rpy=3.1416 -1.57 0 -> xyz=0 0 -0.31 rpy=-1.5708 0 0
- joint laser_joint: parent base_link -> sara_base
- joint shoulderRot_joint: origin xyz=0.085 0 0 rpy=0 1.57 0 -> xyz=-0.085 0 0 rpy=1.5708 0 1.5708
- joint shoulder_joint: origin xyz=0.085 0 0 rpy=1.57 0 1.57 -> xyz=0 -0.085 0 rpy=-1.57 0 0
- joint sternoclavicular_joint: origin xyz=0 -0.145 0 rpy=-1.57 0 -1.57 -> xyz=0 -0.145 0 rpy=0 -1.57 0

Commit message: update joints orientation

File: src/sara_description/urdf/sara.urdf (robot description, URDF)
Before this commit: robot sara, 12 links, 11 joints
Links:
- link spine_link: geometry collision cylinder length=0.9 radius=0.04; visual cylinder length=0.9 radius=0.04
- link torso_link: geometry collision box size=0.04 0.38 0.075; collision box size=0.18 0.18 0.28
Joints:
- joint elbow_joint: limit lower=-2.23 upper=2 effort=1000.0 velocity=0.5 -> lower=-2.20 upper=1.90 effort=1000.0 velocity=0.5
- joint shoulderRot_joint: limit lower=-3.1416 upper=3.1416 effort=1000.0 velocity=0.5 -> lower=-2.14 upper=1.00 effort=1000.0 velocity=0.5
- joint shoulder_joint: limit lower=-3.1416 upper=3.1416 effort=1000.0 velocity=0.5 -> lower=-3.29 upper=0.37 effort=1000.0 velocity=0.5
- joint sternoclavicular_joint: limit lower=-1.57 upper=1.57 effort=1000.0 velocity=0.5 -> lower=-0.18 upper=1.21 effort=1000.0 velocity=0.5
